File: kicad/EasyFlyback2.kicad_pcb (KiCad board)
At the start: 4 copper layers, 59.5 x 72 mm, 47 parts, among them J2 Screw_Terminal_01x02, J3 Screw_Terminal_01x02, J4 AudioJack2, Q2 NMOS, Q3 BC327, SW1 SW_Push, U1 LM311, U2 NE555D

Commit message: Add files via upload
Parts:
- moved C6 0.84 mm to (162.1, 116.8)
Routing:
- net GND: track 170.6 -> 4.39 mm, vias 9 -> 0
- net +12V: track 32.1 -> 0.23 mm, vias 4 -> 0
